Commit message: fixed bugs

File: urdf/lucrezio.urdf (copy).xacro (robot description, xacro)
@@ -159,7 +159,7 @@
   <!-- HOKUYO SENSOR -->
   <gazebo reference="laser_link">
-    <sensor type="ray" name="head_hokuyo_sensor">
+    <sensor type="gpu_ray" name="head_hokuyo_sensor">
       <pose>0 0 0 0 0 0</pose>
-      <visualize>true</visualize>
+      <visualize>false</visualize>
       <update_rate>40</update_rate>
       <ray>
@@ -175,5 +175,5 @@
           <min>0.02</min>
           <max>10.0</max>
-          <resolution>0.1</resolution>
+          <resolution>0.01</resolution>
         </range>
         <noise>
@@ -183,5 +183,5 @@
         </noise>
       </ray>
-      <plugin name="gazebo_ros_head_hokuyo_controller" filename="libgazebo_ros_laser.so">
+      <plugin name="gazebo_ros_head_hokuyo_controller" filename="libgazebo_ros_gpu_laser.so">
         <topicName>/scan</topicName>
         <frameName>laser_link</frameName>

File: urdf/lucrezio_with_logical.urdf.xacro (robot description, xacro)
@@ -47,11 +47,23 @@
   <gazebo>
   <plugin name="ground_truth" filename="libgazebo_ros_p3d.so">
-    <frameName>map</frameName>
+    <alwaysOn>true</alwaysOn>
+     <frameName>camera_link</frameName>
+    <bodyName>camera_link</bodyName>
+    <topicName>/odom</topicName>
+    <updateRate>100.0</updateRate>
+  </plugin>
+  </gazebo> -->
+  <!--
+<gazebo>
+  <controller:ros_p3d name="my_box_controller" plugin="libgazebo_ros_p3d.so">
+    <alwaysOn>true</alwaysOn>
+    <updateRate>100.0</updateRate>
     <bodyName>base_link</bodyName>
-    <topicName>sbrodom</topicName>
-    <updateRate>30.0</updateRate>
-  </plugin>
-  </gazebo>
-  -->
+    <topicName>my_box_pose_ground_truth</topicName>
+    <gaussianNoise>0.0</gaussianNoise>
+    <frameName>base_link</frameName>
+    <interface:position name="my_box_p3d_position_iface" />
+  </controller:ros_p3d>
+  </gazebo> -->
   <!-- LEFT WHEEL -->
   <link name="left_wheel">
@@ -171,13 +183,13 @@
     <sensor type="gpu_ray" name="head_hokuyo_sensor">
       <pose>0 0 0 0 0 0</pose>
-      <visualize>false</visualize>
+      <visualize>true</visualize>
       <update_rate>40</update_rate>
       <ray>
         <scan>
           <horizontal>
-            <samples>1024</samples>
+            <samples>512</samples>
             <resolution>1</resolution>
-            <min_angle>-3.14159</min_angle>
-            <max_angle>3.14159</max_angle>
+            <min_angle>-1.571</min_angle>
+            <max_angle>1.571</max_angle>
           </horizontal>
         </scan>
@@ -310,5 +322,6 @@
   <gazebo>
     <plugin name="gazebo_ros_control" filename="libgazebo_ros_control.so">
-      <robotNamespace>/</robotNamespace>
+        <robotNamespace>/</robotNamespace>
+        <legacyModeNS>true</legacyModeNS>
     </plugin>
   </gazebo>

File: urdf/test.urdf.xacro (robot description, xacro)
@@ -7,5 +7,5 @@
   <xacro:property name="wheel_length" value="0.05" />
   <xacro:property name="wheel_radius" value="0.1" />
-  <xacro:property name="camera_link" value="0.05" />
+  <xacro:property name="camera_size" value="0.05" />
   <xacro:property name="camera_name" value="xtion" />
   <xacro:property name="M_PI" value="3.1415926535897931" />
@@ -44,4 +44,14 @@
     <material>Gazebo/Black</material>
   </gazebo>
+  <!-- Ground Truth Pose Publisher Plug-in
+  <gazebo>
+  <plugin name="ground_truth" filename="libgazebo_ros_p3d.so">
+    <frameName>map</frameName>
+    <bodyName>base_link</bodyName>
+    <topicName>sbrodom</topicName>
+    <updateRate>30.0</updateRate>
+  </plugin>
+  </gazebo>
+  -->
   <!-- LEFT WHEEL -->
   <link name="left_wheel">
@@ -159,5 +169,5 @@
   <!-- HOKUYO SENSOR -->
   <gazebo reference="laser_link">
-    <sensor type="ray" name="head_hokuyo_sensor">
+    <sensor type="gpu_ray" name="head_hokuyo_sensor">
       <pose>0 0 0 0 0 0</pose>
       <visualize>true</visualize>
@@ -168,12 +178,12 @@
             <samples>1024</samples>
             <resolution>1</resolution>
-            <min_angle>-1.57</min_angle>
-            <max_angle>1.57</max_angle>
+            <min_angle>-3.14159</min_angle>
+            <max_angle>3.14159</max_angle>
           </horizontal>
         </scan>
         <range>
-          <min>0.02</min>
-          <max>10.0</max>
-          <resolution>0.1</resolution>
+          <min>0.10</min>
+          <max>15.0</max>
+          <resolution>0.01</resolution>
         </range>
         <noise>
@@ -183,5 +193,5 @@
         </noise>
       </ray>
-      <plugin name="gazebo_ros_head_hokuyo_controller" filename="libgazebo_ros_laser.so">
+      <plugin name="gazebo_ros_head_hokuyo_controller" filename="libgazebo_ros_gpu_laser.so">
         <topicName>/scan</topicName>
         <frameName>laser_link</frameName>
@@ -194,11 +204,11 @@
       <origin xyz="0 0 0" rpy="0 0 0"/>
       <geometry>
-    <box size="${camera_link} ${camera_link} ${camera_link}"/>
-      </geometry>
-    </collision>
-    <visual>
-      <origin xyz="0 0 0" rpy="0 0 0"/>
-      <geometry>
-    <box size="${camera_link} ${camera_link} ${camera_link}"/>
+    <box size="${camera_size} ${camera_size} ${camera_size}"/>
+      </geometry>
+    </collision>
+    <visual>
+      <origin xyz="0 0 0" rpy="0 0 0"/>
+      <geometry>
+    <box size="${camera_size} ${camera_size} ${camera_size}"/>
       </geometry>
       <material name="red"/>
@@ -213,23 +223,18 @@
   <joint name="camera_joint" type="continuous">
     <axis xyz="0 1 0" />
-    <origin xyz="0 0 1.0" rpy="0 0 0"/>
+    <origin xyz="0 0 0.5" rpy="0 0 0"/>
     <parent link="base_link"/>
     <child link="camera_link"/>
   </joint>
-<!--
-  <gazebo reference="camera_joint">
-    <preserveFixedJoint>true</preserveFixedJoint>
-  </gazebo>"
--->
   <!-- XTION SENSOR -->
   <gazebo reference="camera_link">
     <sensor type="depth" name="rgbd_camera">
       <always_on>true</always_on>
-      <update_rate>20.0</update_rate>
+      <update_rate>30.0</update_rate>
       <camera>
         <horizontal_fov>${60.0*M_PI/180.0}</horizontal_fov>
         <image>
-          <width>320</width>
-          <height>240</height>
+          <width>640</width>
+          <height>480</height>
           <format>R8G8B8</format>
         </image>
@@ -242,5 +247,5 @@
         <cameraName>camera</cameraName>
           <alwaysOn>true</alwaysOn>
-          <updateRate>10</updateRate>
+          <updateRate>30</updateRate>
           <imageTopicName>rgb/image_raw</imageTopicName>
           <depthImageTopicName>depth/image_raw</depthImageTopicName>
@@ -259,4 +264,47 @@
     </sensor>
   </gazebo>
+  <!-- LOGICAL CAMERA -->
+  <link name="logical_camera_link">
+    <collision>
+      <origin xyz="0 0 0" rpy="0 0 0"/>
+      <geometry>
+    <box size="${camera_size} ${camera_size} ${camera_size}"/>
+      </geometry>
+    </collision>
+    <visual>
+      <origin xyz="0 0 0" rpy="0 0 0"/>
+      <geometry>
+    <box size="${camera_size} ${camera_size} ${camera_size}"/>
+      </geometry>
+      <material name="red"/>
+    </visual>
+    <inertial>
+      <mass value="1e-5" />
+      <origin xyz="0 0 0" rpy="0 0 0"/>
+      <inertia ixx="1e-6" ixy="0" ixz="0" iyy="1e-6" iyz="0" izz="1e-6" />
+    </inertial>
+  </link>
+  <!-- LOGICAL CAMERA JOINT -->
+  <joint name="logical_camera_joint" type="continuous">
+    <axis xyz="0 1 0" />
+    <origin xyz="0 0 0.5" rpy="0 0 0"/>
+    <parent link="base_link"/>
+    <child link="logical_camera_link"/>
+  </joint>
+  <!-- LOGICAL CAMERA SENSOR -->
+  <gazebo reference="logical_camera_link">
+      <sensor name="logical_camera" type="logical_camera">
+        <plugin name="logical_camera_plugin" filename="liblogical_camera_plugin.so"/>
+          <logical_camera>
+            <near>0.02</near>
+            <far>8.0</far>
+            <horizontal_fov>${60.0*M_PI/180.0}</horizontal_fov>
+            <aspect_ratio>1.778</aspect_ratio>
+          </logical_camera>
+          <visualize>false</visualize>
+          <always_on>true</always_on>
+          <update_rate>20</update_rate>
+      </sensor>
+  </gazebo>
   <!-- Gazebo plugin for ROS Control -->
   <gazebo>
