Commit message: bug kill

File: urdf/lucrezio_with_logical_noLaser.urdf.xacro (robot description, xacro)
@@ -152,4 +152,63 @@
     </joint>
   </transmission>
+  <!-- LASER -->
+  <link name="laser_link">
+    <collision>
+      <origin xyz="0 0 0" rpy="0 0 0" />
+      <geometry>
+        <box size="0.1 0.1 0.1" />
+      </geometry>
+    </collision>
+    <visual>
+      <origin xyz="0 0 0" rpy="0 0 0" />
+      <geometry>
+        <mesh filename="package://lucrezio_simulation_environments/meshes/hokuyo.dae" />
+      </geometry>
+    </visual>
+    <inertial>
+      <mass value="1e-5" />
+      <origin xyz="0 0 0" rpy="0 0 0"/>
+      <inertia ixx="1e-6" ixy="0" ixz="0" iyy="1e-6" iyz="0" izz="1e-6" />
+    </inertial>
+  </link>
+  <!-- LASER JOINT -->
+  <joint name="laser_joint" type="fixed">
+    <axis xyz="0 1 0" />
+    <origin xyz="0.1 0 0.1" rpy="0 0 0" />
+    <parent link="base_link" />
+    <child  link="laser_link" />
+  </joint>
+  <!-- HOKUYO SENSOR -->
+  <gazebo reference="laser_link">
+    <sensor type="gpu_ray" name="head_hokuyo_sensor">
+      <pose>0 0 0 0 0 0</pose>
+      <visualize>true</visualize>
+      <update_rate>40</update_rate>
+      <ray>
+        <scan>
+          <horizontal>
+            <samples>8</samples>
+            <resolution>1</resolution>
+            <min_angle>-1.0</min_angle>
+            <max_angle>1.0</max_angle>
+          </horizontal>
+        </scan>
+        <range>
+          <min>0.10</min>
+          <max>5.0</max>
+          <resolution>0.1</resolution>
+        </range>
+        <noise>
+          <type>gaussian</type>
+          <mean>0.0</mean>
+          <stddev>0.0</stddev>
+        </noise>
+      </ray>
+      <plugin name="gazebo_ros_head_hokuyo_controller" filename="libgazebo_ros_gpu_laser.so">
+        <topicName>/scan</topicName>
+        <frameName>laser_link</frameName>
+      </plugin>
+    </sensor>
+  </gazebo>
   <!-- CAMERA -->
   <link name="camera_link">

Commit message: tilting problem fix

File: urdf/lucrezio_with_logical_noLaser.urdf.xacro (robot description, xacro)
@@ -40,6 +40,4 @@
   </link>
   <gazebo reference="base_link">
-    <mu1>0.0</mu1>
-    <mu2>0.0</mu2>
     <material>Gazebo/Black</material>
   </gazebo>
@@ -88,5 +86,5 @@
     <mu1 value="200.0"/>
     <mu2 value="100.0"/>
-    <kp value="10000000.0" />
+    <kp value="10000000000.0" />
     <kd value="1.0" />
     <material>Gazebo/Grey</material>
@@ -131,5 +129,5 @@
     <mu1 value="200.0"/>
     <mu2 value="100.0"/>
-    <kp value="10000000.0" />
+    <kp value="10000000000.0" />
     <kd value="1.0" />
     <material>Gazebo/Grey</material>
@@ -233,5 +231,5 @@
   </link>
   <!-- CAMERA JOINT -->
-  <joint name="camera_joint" type="continuous">
+  <joint name="camera_joint" type="fixed">
     <axis xyz="0 1 0" />
     <origin xyz="0 0 0.5" rpy="0 0 0"/>
@@ -298,5 +296,5 @@
   </link>
   <!-- LOGICAL CAMERA JOINT -->
-  <joint name="logical_camera_joint" type="continuous">
+  <joint name="logical_camera_joint" type="fixed">
     <axis xyz="0 1 0" />
     <origin xyz="0 0 0.5" rpy="0 0 0"/>
