Commit message: setup

File: urdf/lucrezio_with_logical.urdf.xacro (robot description, xacro)
@@ -160,10 +160,10 @@
       </geometry>
     </collision>
-    <visual>
+    <!--visual>
       <origin xyz="0 0 0" rpy="0 0 0" />
       <geometry>
         <mesh filename="package://lucrezio_simulation_environments/meshes/hokuyo.dae" />
       </geometry>
-    </visual>
+    </visual-->
     <inertial>
       <mass value="1e-5" />
@@ -184,12 +184,12 @@
       <pose>0 0 0 0 0 0</pose>
       <visualize>true</visualize>
-      <update_rate>40</update_rate>
+      <update_rate>20</update_rate>
       <ray>
         <scan>
           <horizontal>
-            <samples>512</samples>
+            <samples>1024</samples>
             <resolution>1</resolution>
-            <min_angle>-1.571</min_angle>
-            <max_angle>1.571</max_angle>
+            <min_angle>-3.13</min_angle>
+            <max_angle>3.14</max_angle>
           </horizontal>
         </scan>
@@ -213,10 +213,10 @@
   <!-- CAMERA -->
   <link name="camera_link">
-    <collision>
+    <!--collision>
       <origin xyz="0 0 0" rpy="0 0 0"/>
       <geometry>
     <box size="${camera_size} ${camera_size} ${camera_size}"/>
       </geometry>
-    </collision>
+    </collision-->
     <visual>
       <origin xyz="0 0 0" rpy="0 0 0"/>

File: urdf/lucrezio_with_logical_noLaser.urdf.xacro (robot description, xacro)
@@ -160,10 +160,10 @@
       </geometry>
     </collision>
-    <visual>
+    <!--visual>
       <origin xyz="0 0 0" rpy="0 0 0" />
       <geometry>
         <mesh filename="package://lucrezio_simulation_environments/meshes/hokuyo.dae" />
       </geometry>
-    </visual>
+    </visual-->
     <inertial>
       <mass value="1e-5" />
@@ -184,5 +184,5 @@
       <pose>0 0 0 0 0 0</pose>
       <visualize>true</visualize>
-      <update_rate>40</update_rate>
+      <update_rate>4</update_rate>
       <ray>
         <scan>

Commit message: add environments and models

File: urdf/lucrezio_with_logical.urdf.xacro (robot description, xacro)
@@ -17,9 +17,9 @@
       </geometry>
     </visual>
-    <collision>
+    <!--collision>
       <geometry>
         <box size="${base_length} ${base_width} ${base_height}"/>
       </geometry>
-    </collision>
+    </collision-->
     <visual>
       <origin xyz="-${base_length/2 - base_height/2} 0 -${base_height/2}" rpy="0 0 0" />
@@ -86,8 +86,8 @@
   </link>
   <gazebo reference="left_wheel">
-    <mu1 value="1.5"/>
-    <mu2 value="1.5"/>
+    <mu1 value="200.0"/>
+    <mu2 value="100.0"/>
     <kp value="10000000.0" />
-    <kd value="100.0" />
+    <kd value="1.0" />
     <material>Gazebo/Grey</material>
   </gazebo>
@@ -129,8 +129,8 @@
   </link>
   <gazebo reference="right_wheel">
-    <mu1 value="1.5"/>
-    <mu2 value="1.5"/>
+    <mu1 value="200.0"/>
+    <mu2 value="100.0"/>
     <kp value="10000000.0" />
-    <kd value="100.0" />
+    <kd value="1.0" />
     <material>Gazebo/Grey</material>
   </gazebo>
@@ -154,10 +154,10 @@
   <!-- LASER -->
   <link name="laser_link">
-    <collision>
+    <!--collision>
       <origin xyz="0 0 0" rpy="0 0 0" />
       <geometry>
         <box size="0.1 0.1 0.1" />
       </geometry>
-    </collision>
+    </collision-->
     <!--visual>
       <origin xyz="0 0 0" rpy="0 0 0" />
@@ -175,5 +175,5 @@
   <joint name="laser_joint" type="fixed">
     <axis xyz="0 1 0" />
-    <origin xyz="0.1 0 0.1" rpy="0 0 0" />
+    <origin xyz="0.1 0 -0.05" rpy="0 0 0" />
     <parent link="base_link" />
     <child  link="laser_link" />
@@ -181,21 +181,29 @@
   <!-- HOKUYO SENSOR -->
   <gazebo reference="laser_link">
-    <sensor type="ray" name="head_hokuyo_sensor">
+    <sensor type="ray" name="head_hokuyo_sensor"> <!-- type="gpu_ray" -->
       <pose>0 0 0 0 0 0</pose>
-      <visualize>true</visualize>
-      <update_rate>20</update_rate>
+      <visualize>false</visualize>
+      <update_rate>40</update_rate>
       <ray>
+        <!--scan>
+          <horizontal>
+            <samples>512</samples>
+            <resolution>1</resolution>
+            <min_angle>${-(60.0*M_PI/360.0)}</min_angle>
+            <max_angle>${+(60.0*M_PI/360.0)}</max_angle>
+          </horizontal>
+        </scan-->
         <scan>
           <horizontal>
-            <samples>1024</samples>
+            <samples>512</samples>
             <resolution>1</resolution>
-            <min_angle>-3.14</min_angle>
-            <max_angle>3.13</max_angle>
+            <min_angle>-1.571</min_angle>
+            <max_angle>1.571</max_angle>
           </horizontal>
         </scan>
         <range>
-          <min>0.2</min>
-          <max>12.0</max>
-          <resolution>0.1</resolution>
+          <min>0.20</min>
+          <max>15.0</max>
+          <resolution>0.01</resolution>
         </range>
         <noise>
@@ -205,5 +213,5 @@
         </noise>
       </ray>
-      <plugin name="gazebo_ros_head_hokuyo_controller" filename="libgazebo_ros_laser.so">
+      <plugin name="gazebo_ros_head_hokuyo_controller" filename="libgazebo_ros_laser.so"> <!-- "libgazebo_ros_gpu_laser.so -->
         <topicName>/scan</topicName>
         <frameName>laser_link</frameName>
@@ -233,5 +241,5 @@
   </link>
   <!-- CAMERA JOINT -->
-  <joint name="camera_joint" type="continuous">
+  <joint name="camera_joint" type="fixed">
     <axis xyz="0 1 0" />
     <origin xyz="0 0 0.5" rpy="0 0 0"/>
@@ -298,5 +306,5 @@
   </link>
   <!-- LOGICAL CAMERA JOINT -->
-  <joint name="logical_camera_joint" type="continuous">
+  <joint name="logical_camera_joint" type="fixed">
     <axis xyz="0 1 0" />
     <origin xyz="0 0 0.5" rpy="0 0 0"/>
@@ -323,5 +331,4 @@
     <plugin name="gazebo_ros_control" filename="libgazebo_ros_control.so">
         <robotNamespace>/</robotNamespace>
-        <legacyModeNS>true</legacyModeNS>
     </plugin>
   </gazebo>

File: urdf/lucrezio_with_logical_noLaser.urdf.xacro (robot description, xacro)
@@ -84,6 +84,6 @@
   </link>
   <gazebo reference="left_wheel">
-    <mu1 value="200.0"/>
-    <mu2 value="100.0"/>
+    <mu1 value="1.0"/>
+    <mu2 value="1.0"/>
     <kp value="10000000000.0" />
     <kd value="1.0" />
@@ -127,6 +127,6 @@
   </link>
   <gazebo reference="right_wheel">
-    <mu1 value="200.0"/>
-    <mu2 value="100.0"/>
+    <mu1 value="1.0"/>
+    <mu2 value="1.0"/>
     <kp value="10000000000.0" />
     <kd value="1.0" />
